File: hardware/bGeigieNanoKit/bGeigieNanoKit.sch (EAGLE design)
At the start: 35 parts, among them T1 2SC1815

Commit message: rc1
Parts:
- removed ALARM: RED, adafruit:LED3MM
- removed CN1: (no value), microbuilder:AUDIO_STEREOJACK
- removed U$1: OPENLOG, open_hw_sockets:OPENLOG
- removed U$2: FIO_SOCKETBOT, open_hw_sockets:FIO_SOCKETBOT
- removed U$3: GPS, open_hw_sockets:ULTIMATE_GPSTOP
- removed U$5: LCD, open_hw_sockets:SSD1306_128X64_LCD_MIN
- added FIO: FIO_SOCKETBOT, open_hw_sockets:FIO_SOCKETBOT
- added GPS: ULTIMATE_GPSTOP, open_hw_sockets:ULTIMATE_GPSTOP
- added JP2: (no value), SparkFun:M02PTH
- added JP3, JP5: M01PTH, SparkFun:M01PTH
- added JP4: (no value), SparkFun:M081X08
- added JP6: (no value), SparkFun:JUMPER-2SMD-NO
- added JP7: (no value), microbuilder:JUMPER2
- added JP8: (no value), SparkFun:M06SIP
- added LCD: SSD1306_128X64_V2_LCD1.3IN_TOP, open_hw_sockets:SSD1306_128X64_V2_LCD1.3IN_TOP
- added LCD2: SSD1306_128X64_V2_LCD0.96IN_MIN, open_hw_sockets:SSD1306_128X64_V2_LCD0.96IN_MIN
- added LOG/ALARM: RED, adafruit:LED3MM
- added OPENLOG: OPENLOG, open_hw_sockets:OPENLOG
- JP1: device con-lstb:MA03-1 -> pinhead:PINHD-1X3/90
Connections:
- new net N$31: CHARGE.C, R11.2
- new net N$32: R7.1, SG1.1, SW1.4
- new net N$33: FIO.A4, JP4.5
- new net N$34: FIO.A3, JP4.4
- new net N$35: FIO.A2, JP4.3
- new net N$36: FIO.A1, JP4.2
- new net N$37: FIO.DTR@1, JP8.6
- new net N$38: FIO.TXO, JP8.5
- new net N$39: FIO.RXI, JP8.4
- new net N$40: FIO.AREF, JP8.2
- new net VGPS: GPS.VBAT, JP6.2
- net GND: now also FIO.GND@1, FIO.GND@2, FIO.GND@3, FIO.GND@4, GPS.GND, JP1.3, JP2.2, JP7.2, JP8.1, LCD.GND, LCD2.GND, LOG/ALARM.C, OPENLOG.GND@1, OPENLOG.GND@2, U$4.P$1; no longer ALARM.C, CHARGE.C, CN1.1, JP1.1, U$1.GND@1, U$1.GND@2, U$2.GND@1, U$2.GND@2, U$2.GND@3, U$2.GND@4, U$3.GND, U$4.P$3, U$5.GND
- net N$1: now also FIO.D9, LCD.DATA, LCD2.DATA; no longer U$2.D9, U$5.D1/DATA
- net N$10: now also FIO.D4, OPENLOG.DTR; no longer U$1.DTR, U$2.D4
- net N$11: now also FIO.A0, JP4.1; no longer U$2.A0
- net N$12: now also FIO.SW+; no longer U$2.SW+
- net N$13: now also FIO.SW-; no longer U$2.SW-
- net N$14: now also FIO.A7, JP4.8; no longer U$2.A7
- net N$15: now also FIO.A6, JP4.7; no longer U$2.A2
- net N$16: now also LOG/ALARM.A, SW1.3; no longer ALARM.A, SW1.1
- net N$17: now also SW1.2; no longer SW1.4
- net N$18: now also FIO.D2; no longer U$2.D2
- net N$2: now also FIO.D10, LCD.CLK, LCD2.CLK; no longer U$2.D10, U$5.D0/CLK
- net N$21: now also FIO.A5, JP4.6; no longer R7.1, SG1.1, SW1.2
- net N$25: now also JP2.1; no longer CN1.2
- net N$29: now also JP7.1; no longer CHARGE.A
- net N$3: now also FIO.D11, LCD.DC, LCD2.DC; no longer U$2.D11, U$5.D/C
- net N$30: now also FIO.D3; no longer U$2.D3
- net N$4: now also FIO.D12, LCD.CS, LCD2.CS; no longer U$2.D12, U$5.CS
- net N$5: now also FIO.D13, LCD.RST, LCD2.RST; no longer U$2.D13, U$5.RES
- net N$6: now also FIO.D8, GPS.TX; no longer U$2.D8, U$3.TX
- net N$7: now also FIO.D7, GPS.RX; no longer U$2.D7, U$3.RX
- net N$8: now also FIO.D6, OPENLOG.TXO; no longer U$1.TXO, U$2.D6
- net N$9: now also FIO.D5, OPENLOG.RXI; no longer U$1.RXI, U$2.D5
- net VBATT: now also FIO.VBATT, JP6.1; no longer U$2.VBATT
- net VCC: now also FIO.3V3@1, FIO.3V3@2, GPS.VIN, JP1.1, JP8.3, LCD.VIN, LCD2.VIN, OPENLOG.VCC, SW1.1; no longer JP1.3, SW1.3, U$1.VCC, U$2.3V3@1, U$2.3V3@2, U$3.VIN, U$5.VBAT, U$5.VDD
- net VIN: now also CHARGE.A, FIO.VIN; no longer R11.2, U$2.VIN
Other:
- moved on the sheet: C1, C2, C3, CHARGE, COUNT, D1, R1, R10, R11, R12, R2, R3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

Commit message: commiting all changes for what should be Release v1.0
Parts:
- removed JP3, JP5: M01PTH, SparkFun:M01PTH
- S1: device adafruit:EG1218S -> open_hw_sockets:EG1218S
Changed lines of the file:
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@@
 <grid distance="0.1" unitdist="inch" unit="inch" style="lines" multiple="1" display="no" altdistance="0.01" altunitdist="inch" altunit="inch"/>
 <layers>
-<layer number="1" name="Top" color="4" fill="1" visible="yes" active="no"/>
-<layer number="2" name="Route2" color="1" fill="3" visible="yes" active="no"/>
-<layer number="3" name="Route3" color="4" fill="3" visible="yes" active="no"/>
-<layer number="14" name="Route14" color="1" fill="6" visible="yes" active="no"/>
-<layer number="15" name="Route15" color="4" fill="6" visible="yes" active="no"/>
-<layer number="16" name="Bottom" color="1" fill="1" visible="yes" active="no"/>
-<layer number="17" name="Pads" color="2" fill="1" visible="yes" active="no"/>
-<layer number="18" name="Vias" color="2" fill="1" visible="yes" active="no"/>
-<layer number="19" name="Unrouted" color="6" fill="1" visible="yes" active="no"/>
-<layer number="20" name="Dimension" color="15" fill="1" visible="yes" active="no"/>
-<layer number="21" name="tPlace" color="14" fill="1" visible="yes" active="no"/>
-<layer number="22" name="bPlace" color="13" fill="1" visible="yes" active="no"/>
-<layer number="23" name="tOrigins" color="15" fill="1" visible="yes" active="no"/>
-<layer number="24" name="bOrigins" color="15" fill="1" visible="yes" active="no"/>
-<layer number="25" name="tNames" color="7" fill="1" visible="yes" active="no"/>
-<layer number="26" name="bNames" color="7" fill="1" visible="yes" active="no"/>
-<layer number="27" name="tValues" color="7" fill="1" visible="yes" active="no"/>
-<layer number="28" name="bValues" color="7" fill="1" visible="yes" active="no"/>
+<layer number="1" name="Top" color="4" fill="1" visible="no" active="no"/>
+<layer number="2" name="Route2" color="1" fill="3" visible="no" active="no"/>
+<layer number="3" name="Route3" color="4" fill="3" visible="no" active="no"/>
+<layer number="14" name="Route14" color="1" fill="6" visible="no" active="no"/>
+<layer number="15" name="Route15" color="4" fill="6" visible="no" active="no"/>
+<layer number="16" name="Bottom" color="1" fill="1" visible="no" active="no"/>
+<layer number="17" name="Pads" color="2" fill="1" visible="no" active="no"/>
+<layer number="18" name="Vias" color="2" fill="1" visible="no" active="no"/>
+<layer number="19" name="Unrouted" color="6" fill="1" visible="no" active="no"/>
+<layer number="20" name="Dimension" color="15" fill="1" visible="no" active="no"/>
+<layer number="21" name="tPlace" color="14" fill="1" visible="no" active="no"/>
+<layer number="22" name="bPlace" color="13" fill="1" visible="no" active="no"/>
+<layer number="23" name="tOrigins" color="15" fill="1" visible="no" active="no"/>
+<layer number="24" name="bOrigins" color="15" fill="1" visible="no" active="no"/>
+<layer number="25" name="tNames" color="7" fill="1" visible="no" active="no"/>
+<layer number="26" name="bNames" color="7" fill="1" visible="no" active="no"/>
+<layer number="27" name="tValues" color="7" fill="1" visible="no" active="no"/>
+<layer number="28" name="bValues" color="7" fill="1" visible="no" active="no"/>
 <layer number="29" name="tStop" color="7" fill="3" visible="no" active="no"/>
 <layer number="30" name="bStop" color="7" fill="6" visible="no" active="no"/>
@@
 <layer number="35" name="tGlue" color="7" fill="4" visible="no" active="no"/>
 <layer number="36" name="bGlue" color="7" fill="5" visible="no" active="no"/>
-<layer number="37" name="tTest" color="7" fill="1" visible="yes" active="no"/>
-<layer number="38" name="bTest" color="7" fill="1" visible="yes" active="no"/>
+<layer number="37" name="tTest" color="7" fill="1" visible="no" active="no"/>
+<layer number="38" name="bTest" color="7" fill="1" visible="no" active="no"/>
 <layer number="39" name="tKeepout" color="4" fill="11" visible="no" active="no"/>
 <layer number="40" name="bKeepout" color="1" fill="11" visible="no" active="no"/>
@@
 <layer number="44" name="Drills" color="7" fill="1" visible="no" active="no"/>
 <layer number="45" name="Holes" color="7" fill="1" visible="no" active="no"/>
-<layer number="46" name="Milling" color="3" fill="1" visible="yes" active="no"/>
-<layer number="47" name="Measures" color="7" fill="1" visible="yes" active="no"/>
-<layer number="48" name="Document" color="7" fill="1" visible="yes" active="no"/>
-<layer number="49" name="Reference" color="7" fill="1" visible="yes" active="no"/>
-<layer number="50" name="dxf" color="7" fill="1" visible="yes" active="no"/>
-<layer number="51" name="tDocu" color="7" fill="1" visible="yes" active="no"/>
-<layer number="52" name="bDocu" color="7" fill="1" visible="yes" active="no"/>
-<layer number="53" name="tGND_GNDA" color="7" fill="9" visible="yes" active="no"/>
-<layer number="54" name="bGND_GNDA" color="1" fill="9" visible="yes" active="no"/>
-<layer number="56" name="wert" color="7" fill="1" visible="yes" active="no"/>
+<layer number="46" name="Milling" color="3" fill="1" visible="no" active="no"/>
+<layer number="47" name="Measures" color="7" fill="1" visible="no" active="no"/>
+<layer number="48" name="Document" color="7" fill="1" visible="no" active="no"/>
+<layer number="49" name="Reference" color="7" fill="1" visible="no" active="no"/>
+<layer number="50" name="dxf" color="7" fill="1" visible="no" active="no"/>
+<layer number="51" name="tDocu" color="7" fill="1" visible="no" active="no"/>
+<layer number="52" name="bDocu" color="7" fill="1" visible="no" active="no"/>
+<layer number="53" name="tGND_GNDA" color="7" fill="9" visible="no" active="no"/>
+<layer number="54" name="bGND_GNDA" color="1" fill="9" visible="no" active="no"/>
+<layer number="56" name="wert" color="7" fill="1" visible="no" active="no"/>
 <layer number="91" name="Nets" color="2" fill="1" visible="yes" active="yes"/>
 <layer number="92" name="Busses" color="1" fill="1" visible="yes" active="yes"/>
@@
 <part name="JP1" library="pinhead" deviceset="PINHD-1X3" device="/90"/>
 <part name="S5" library="SparkFun" deviceset="SWITCH-MOMENTARY-2" device="PTH" value=""/>
-<part name="S1" library="adafruit" deviceset="EG1218" device="S"/>
+<part name="S1" library="open_hw_sockets" deviceset="EG1218" device="S"/>
 <part name="SG1" library="SparkFun" deviceset="BUZZER" device="PTH" value="BUZZER"/>
 <part name="FIO" library="open_hw_sockets" deviceset="FIO_SOCKET" device="BOT" value="FIO_SOCKETBOT"/>
@@
 <part name="LCD" library="open_hw_sockets" deviceset="SSD1306_128X64_V2_LCD" device="1.3IN_TOP" value="SSD1306_128X64_V2_LCD1.3IN_TOP"/>
 <part name="JP4" library="SparkFun" deviceset="M08" device="1X08"/>
-<part name="JP3" library="SparkFun" deviceset="M01" device="PTH"/>
-<part name="JP5" library="SparkFun" deviceset="M01" device="PTH"/>
 <part name="JP6" library="SparkFun" deviceset="JUMPER-2" device="SMD-NO"/>
 <part name="JP7" library="microbuilder" deviceset="JUMPER2" device=""/>
@@
 </instance>
 <instance part="JP4" gate="G$1" x="139.7" y="111.76" rot="MR0"/>
-<instance part="JP3" gate="G$1" x="152.4" y="71.12"/>
-<instance part="JP5" gate="G$1" x="152.4" y="58.42"/>
 <instance part="JP6" gate="A" x="40.64" y="116.84" rot="R270"/>
 <instance part="JP7" gate="A" x="129.54" y="48.26" rot="R270"/>

Commit message: before removing second lcd
Parts:
- JP2: device SparkFun:M02PTH -> microbuilder:HEADER-1X4ROUND
- LCD: value SSD1306_128X64_V2_LCD1.3IN_TOP -> SSD1306_128X64_V2_LCD1.3IN_LEVER; device open_hw_sockets:SSD1306_128X64_V2_LCD1.3IN_TOP -> open_hw_sockets:SSD1306_128X64_V2_LCD1.3IN_LEVER
- LCD2: value SSD1306_128X64_V2_LCD0.96IN_MIN -> SSD1306_128X64_V2_LCD0.96IN_MNT_NOOUT; device open_hw_sockets:SSD1306_128X64_V2_LCD0.96IN_MIN -> open_hw_sockets:SSD1306_128X64_V2_LCD0.96IN_MNT_NOOUT
- R8: value 47k -> 10k
- R9: value 1k -> 2.2k
- S1: device open_hw_sockets:EG1218S -> adafruit:EG1218S
Connections:
- removed net N$21: FIO.A5, JP4.6
- new net N$41: FIO.A7, JP4.8
- net N$14: now also FIO.A5, JP4.6; no longer FIO.A7, JP4.8
- net N$15: no longer R4.1
- net N$33: now also R4.1

Commit message: applied most all changes rc v1.0r2
Parts:
- removed CHARGE: RED, adafruit:LED3MM
- removed JP7: (no value), microbuilder:JUMPER2
- removed LCD2: SSD1306_128X64_V2_LCD0.96IN_MNT_NOOUT, open_hw_sockets:SSD1306_128X64_V2_LCD0.96IN_MNT_NOOUT
- removed R11: 1k, rcl:R-US_0207/10
- C1, C2, C3: device rcl:C-EU050-024X044 -> rcl:C-EU025-024X044
Connections:
- removed net N$29: JP7.1, R11.1
- removed net N$31: CHARGE.C, R11.2
- net GND: no longer JP7.2, LCD2.GND
- net N$1: no longer LCD2.DATA
- net N$2: no longer LCD2.CLK
- net N$3: no longer LCD2.DC
- net N$4: no longer LCD2.CS
- net N$5: no longer LCD2.RST
- net VCC: no longer LCD2.VIN
- net VIN: no longer CHARGE.A
Changed lines of the file:
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@@
 <part name="SUPPLY3" library="supply2" deviceset="GND" device=""/>
 <part name="D1" library="adafruit" deviceset="DIODE" device="DO-1N4148"/>
-<part name="C1" library="rcl" deviceset="C-EU" device="050-024X044" value="0.1uF"/>
-<part name="C2" library="rcl" deviceset="C-EU" device="050-024X044" value="0.1uF"/>
-<part name="C3" library="rcl" deviceset="C-EU" device="050-024X044" value="0.1uF"/>
+<part name="C1" library="rcl" deviceset="C-EU" device="025-024X044" value="0.1uF"/>
+<part name="C2" library="rcl" deviceset="C-EU" device="025-024X044" value="0.1uF"/>
+<part name="C3" library="rcl" deviceset="C-EU" device="025-024X044" value="0.1uF"/>
 <part name="SUPPLY4" library="supply2" deviceset="GND" device=""/>
 <part name="T1" library="transistor" deviceset="2SC1815" device=""/>
@@
 <part name="U$8" library="microbuilder" deviceset="MOUNTINGHOLE" device="3.0THIN"/>
 <part name="U$9" library="microbuilder" deviceset="MOUNTINGHOLE" device="3.0THIN"/>
-<part name="R11" library="rcl" deviceset="R-US_" device="0207/10" value="1k"/>
-<part name="CHARGE" library="adafruit" deviceset="LED" device="3MM" value="RED"/>
-<part name="SUPPLY16" library="supply2" deviceset="GND" device=""/>
 <part name="R12" library="rcl" deviceset="R-US_" device="0207/10" value="1k"/>
 <part name="U$4" library="open_hw_sockets" deviceset="A12JH" device=""/>
@@
 <part name="JP4" library="SparkFun" deviceset="M08" device="1X08"/>
 <part name="JP6" library="SparkFun" deviceset="JUMPER-2" device="SMD-NO"/>
-<part name="JP7" library="microbuilder" deviceset="JUMPER2" device=""/>
-<part name="LCD2" library="open_hw_sockets" deviceset="SSD1306_128X64_V2_LCD" device="0.96IN_MNT_NOOUT" value="SSD1306_128X64_V2_LCD0.96IN_MNT_NOOUT"/>
 <part name="JP8" library="SparkFun" deviceset="M06" device="SIP"/>
 <part name="JP2" library="microbuilder" deviceset="HEADER-1X4" device="ROUND"/>
@@
 <instance part="U$8" gate="G$1" x="233.68" y="30.48"/>
 <instance part="U$9" gate="G$1" x="248.92" y="30.48"/>
-<instance part="R11" gate="G$1" x="114.3" y="48.26" rot="R180"/>
-<instance part="CHARGE" gate="G$1" x="101.6" y="48.26" rot="R90"/>
-<instance part="SUPPLY16" gate="GND" x="119.38" y="43.18"/>
 <instance part="R12" gate="G$1" x="53.34" y="88.9" rot="R90"/>
 <instance part="U$4" gate="G$1" x="165.1" y="137.16"/>
@@
 <instance part="JP4" gate="G$1" x="139.7" y="111.76" rot="MR0"/>
 <instance part="JP6" gate="A" x="40.64" y="116.84" rot="R270"/>
-<instance part="JP7" gate="A" x="129.54" y="48.26" rot="R270"/>
-<instance part="LCD2" gate="G$1" x="38.1" y="149.86" rot="MR180"/>
 <instance part="JP8" gate="G$1" x="127" y="93.98" rot="MR0"/>
 <instance part="JP2" gate="A" x="236.22" y="68.58"/>
@@
 <net name="GND" class="1">
 <segment>
-<wire x1="27.94" y1="157.48" x2="45.72" y2="157.48" width="0.1524" layer="91"/>
 <pinref part="SUPPLY5" gate="GND" pin="GND"/>
 <pinref part="LCD" gate="G$1" pin="GND"/>
-<pinref part="LCD2" gate="G$1" pin="GND"/>
-<wire x1="45.72" y1="157.48" x2="63.5" y2="157.48" width="0.1524" layer="91"/>
-<junction x="45.72" y="157.48"/>
+<wire x1="27.94" y1="157.48" x2="63.5" y2="157.48" width="0.1524" layer="91"/>
 </segment>
 <segment>
@@
 <wire x1="170.18" y1="139.7" x2="167.64" y2="139.7" width="0.1524" layer="91"/>
 </segment>
-<segment>
-<pinref part="SUPPLY16" gate="GND" pin="GND"/>
-<wire x1="127" y1="45.72" x2="119.38" y2="45.72" width="0.1524" layer="91"/>
-<pinref part="JP7" gate="A" pin="2"/>
-</segment>
 </net>
 <net name="VCC" class="1">
@@
 </segment>
 <segment>
-<wire x1="27.94" y1="154.94" x2="45.72" y2="154.94" width="0.1524" layer="91"/>
+<wire x1="27.94" y1="154.94" x2="58.42" y2="154.94" width="0.1524" layer="91"/>
 <label x="50.8" y="154.94" size="1.778" layer="95"/>
 <pinref part="LCD" gate="G$1" pin="VIN"/>
-<pinref part="LCD2" gate="G$1" pin="VIN"/>
-<wire x1="45.72" y1="154.94" x2="58.42" y2="154.94" width="0.1524" layer="91"/>
-<junction x="45.72" y="154.94"/>
 </segment>
 <segment>
@@
 <segment>
 <pinref part="FIO" gate="U$1" pin="VIN"/>
-<label x="96.52" y="50.8" size="1.778" layer="95" rot="R90"/>
-<wire x1="96.52" y1="68.58" x2="96.52" y2="48.26" width="0.1524" layer="91"/>
-<pinref part="CHARGE" gate="G$1" pin="A"/>
-<wire x1="96.52" y1="48.26" x2="99.06" y2="48.26" width="0.1524" layer="91"/>
+<label x="99.06" y="53.34" size="1.778" layer="95"/>
+<wire x1="96.52" y1="68.58" x2="96.52" y2="53.34" width="0.1524" layer="91"/>
+<wire x1="96.52" y1="53.34" x2="106.68" y2="53.34" width="0.1524" layer="91"/>
 </segment>
 </net>
@@
 <wire x1="50.8" y1="111.76" x2="50.8" y2="139.7" width="0.1524" layer="91"/>
 <pinref part="LCD" gate="G$1" pin="DATA"/>
-<wire x1="50.8" y1="139.7" x2="45.72" y2="139.7" width="0.1524" layer="91"/>
-<pinref part="LCD2" gate="G$1" pin="DATA"/>
-<wire x1="45.72" y1="139.7" x2="27.94" y2="139.7" width="0.1524" layer="91"/>
-<junction x="45.72" y="139.7"/>
+<wire x1="50.8" y1="139.7" x2="27.94" y2="139.7" width="0.1524" layer="91"/>
 </segment>
 </net>
@@
 <wire x1="53.34" y1="114.3" x2="53.34" y2="142.24" width="0.1524" layer="91"/>
 <pinref part="LCD" gate="G$1" pin="CLK"/>
-<wire x1="53.34" y1="142.24" x2="45.72" y2="142.24" width="0.1524" layer="91"/>
-<pinref part="LCD2" gate="G$1" pin="CLK"/>
-<wire x1="45.72" y1="142.24" x2="27.94" y2="142.24" width="0.1524" layer="91"/>
-<junction x="45.72" y="142.24"/>
+<wire x1="53.34" y1="142.24" x2="27.94" y2="142.24" width="0.1524" layer="91"/>
 </segment>
 </net>
@@
 <wire x1="55.88" y1="116.84" x2="55.88" y2="144.78" width="0.1524" layer="91"/>
 <pinref part="LCD" gate="G$1" pin="DC"/>
-<wire x1="55.88" y1="144.78" x2="45.72" y2="144.78" width="0.1524" layer="91"/>
-<pinref part="LCD2" gate="G$1" pin="DC"/>
-<wire x1="45.72" y1="144.78" x2="27.94" y2="144.78" width="0.1524" layer="91"/>
-<junction x="45.72" y="144.78"/>
+<wire x1="55.88" y1="144.78" x2="27.94" y2="144.78" width="0.1524" layer="91"/>
 </segment>
 </net>
@@
 <wire x1="58.42" y1="119.38" x2="58.42" y2="149.86" width="0.1524" layer="91"/>
 <pinref part="LCD" gate="G$1" pin="CS"/>
-<wire x1="58.42" y1="149.86" x2="45.72" y2="149.86" width="0.1524" layer="91"/>
-<pinref part="LCD2" gate="G$1" pin="CS"/>
-<wire x1="45.72" y1="149.86" x2="27.94" y2="149.86" width="0.1524" layer="91"/>
-<junction x="45.72" y="149.86"/>
+<wire x1="58.42" y1="149.86" x2="27.94" y2="149.86" width="0.1524" layer="91"/>
 </segment>
 </net>
@@
 <wire x1="60.96" y1="121.92" x2="60.96" y2="147.32" width="0.1524" layer="91"/>
 <pinref part="LCD" gate="G$1" pin="RST"/>
-<wire x1="60.96" y1="147.32" x2="45.72" y2="147.32" width="0.1524" layer="91"/>
-<pinref part="LCD2" gate="G$1" pin="RST"/>
-<wire x1="45.72" y1="147.32" x2="27.94" y2="147.32" width="0.1524" layer="91"/>
-<junction x="45.72" y="147.32"/>
+<wire x1="60.96" y1="147.32" x2="27.94" y2="147.32" width="0.1524" layer="91"/>
 </segment>
 </net>
@@
 </segment>
 </net>
-<net name="N$29" class="0">
-<segment>
-<pinref part="R11" gate="G$1" pin="1"/>
-<wire x1="119.38" y1="48.26" x2="127" y2="48.26" width="0.1524" layer="91"/>
-<pinref part="JP7" gate="A" pin="1"/>
-</segment>
-</net>
-<net name="N$31" class="0">
-<segment>
-<pinref part="CHARGE" gate="G$1" pin="C"/>
-<pinref part="R11" gate="G$1" pin="2"/>
-<wire x1="109.22" y1="48.26" x2="106.68" y2="48.26" width="0.1524" layer="91"/>
-</segment>
-</net>
